Commit message: Used Joint in URDF

File: learnings/my_robot.urdf (robot description, URDF)
Before this commit: robot my_robot, 1 links, 0 joints
Links:
- added link second_link; visual cylinder length=0.2 radius=0.1
- added link third_link; visual box size=0.1 0.1 0.1
Joints:
- added joint base_second_joint: type fixed, parent base_link, child second_link, origin xyz=0.0 0.0 0.2 rpy=0.0 0.0 0.0
- added joint second_third_joint: type fixed, parent second_link, child third_link, origin xyz=0.0 0.0 0.2 rpy=0.0 0.0 0.0

Commit message: Added Sensor Mount in URDF

File: learnings/my_robot.urdf (robot description, URDF)
Before this commit: robot my_robot, 3 links, 2 joints
Links:
- removed link third_link
Joints:
- removed joint second_third_joint
- joint base_second_joint: axis (none) -> 0.0 0.0 1.0; limit (none) -> lower=-1.57 upper=1.57 effort=100.0 velocity=100.0; type fixed -> revolute

Commit message: Done with basic URDF

File: learnings/my_robot.urdf (robot description, URDF)
Before this commit: robot my_robot, 2 links, 1 joints
Links:
- removed link second_link
- added link base_footprint
- added link caster_wheel_link; visual sphere radius=0.05
- added link left_wheel_link; visual cylinder length=0.05 radius=0.1
- added link right_wheel_link; visual cylinder length=0.05 radius=0.1
Joints:
- removed joint base_second_joint
- added joint base_caster_wheel_joint: type fixed, parent base_link, child caster_wheel_link, origin xyz=0.2 0.0 -0.05 rpy=0 0 0, axis 0 1 0
- added joint base_joint: type fixed, parent base_footprint, child base_link, origin xyz=0.0 0.0 0.1 rpy=0.0 0.0 0.0
- added joint base_left_wheel_joint: type continuous, parent base_link, child left_wheel_link, origin xyz=-0.15 0.225 0 rpy=0 0 0, axis 0 1 0
- added joint base_right_wheel_joint: type continuous, parent base_link, child right_wheel_link, origin xyz=-0.15 -0.225 0 rpy=0 0 0, axis 0 1 0
