Commit message: do it later

File: src/my_robot_description/urdf/mobile_base.xacro (robot description, xacro)
@@ -16,4 +16,10 @@
             <material name="blue" />
         </visual>
+        <collision>
+            <geometry>
+                <box size="${base_length} ${base_width} ${base_height}"/>
+            </geometry>
+            <origin xyz="0.0 0.0 ${base_height/2.0}" rpy="0.0 0.0 0.0"/>
+        </collision>
         <xacro:box_inertia m="5.0" x="${base_length}" y="${base_width}" z="${base_height}"
                            o_xyz="0.0 0.0 ${base_height / 2.0}" o_rpy="0.0 0.0 0.0" />
@@ -23,9 +29,15 @@
             <visual>
                 <geometry>
-                    <cylinder radius="${wheel_radius}" length="${wheel_length}"/>
+                    <cylinder radius="${wheel_radius}" />
+                </geometry>
+                <origin xyz="0.0 0.0 0.0" rpy="0.0 0.0 0.0"/>
+               <material name="grey"/>
+            </visual>
+            <collision>
+                <geometry>
+                    <sphere radius="${wheel_radius}" length="${wheel_length}"/>
                 </geometry>
                 <origin xyz="0.0 0.0 0.0" rpy="${pi / 2.0} 0.0 0.0"/>
-               <material name="grey"/>
-            </visual>
+            </collision>
             <xacro:cylinder_inertia m="1.0" r="${wheel_radius}" l="${wheel_length}"
                            o_xyz="0.0 0.0 0.0" o_rpy="${pi / 2.0} 0.0 0.0" />

Commit message: Included GZ launch file

File: src/my_robot_description/urdf/mobile_base.xacro (robot description, xacro)
@@ -29,12 +29,12 @@
             <visual>
                 <geometry>
-                    <cylinder radius="${wheel_radius}" />
+                    <cylinder radius="${wheel_radius}" length="${wheel_length}" />
                 </geometry>
-                <origin xyz="0.0 0.0 0.0" rpy="0.0 0.0 0.0"/>
+                <origin xyz="0.0 0.0 0.0" rpy="${pi / 2.0} 0.0 0.0"/>
                <material name="grey"/>
             </visual>
             <collision>
                 <geometry>
-                    <sphere radius="${wheel_radius}" length="${wheel_length}"/>
+                    <sphere radius="${wheel_radius}"/>
                 </geometry>
                 <origin xyz="0.0 0.0 0.0" rpy="${pi / 2.0} 0.0 0.0"/>
@@ -74,4 +74,10 @@
             <material name="grey"/>
         </visual>
+        <collision>
+            <geometry>
+                <sphere radius="${wheel_radius/2}"/>
+            </geometry>
+            <origin xyz="0.0 0.0 0.0" rpy="0.0 0.0 0.0"/>
+        </collision>
         <xacro:sphere_inertia m="0.5" r="${wheel_radius/2}" o_xyz="0.0 0.0 0.0" o_rpy="0.0 0.0 0.0" />
     </link>
