Commit message: included inertia to box

File: src/my_robot_description/urdf/common_properties.xacro (robot description, xacro)
@@ -8,3 +8,21 @@
         <color rgba="0.5 0.5 0.5 1" />  <!-- Grey -->
     </material>
+    <xacro:macro name="box_inertia" params="m x y z o_xyz o_rpy">
+        <inertial>
+            <mass value="${m}" />
+            <orgin xyz="${o_xyz}" rpy="${o_rpy}" />
+            <inertia ixx="${(m/12)*(y*y + z*z)}" ixy="0" ixz="0"
+                     iyy="${(m/12)*(x*x + z*z)}" iyz="0"
+                     izz="${(m/12)*(x*x + y*y)}" />
+        </inertial>
+    </xacro:macro>
+    <xacro:macro name="wheel_inertia" params="r l w_xyz w_rpy">
+        <inertial>
+            <mass value="${m}" />
+            <orgin xyz="${o_xyz}" rpy="${o_rpy}" />
+            <inertia ixx="${(m/12)*(y*y + z*z)}" ixy="0" ixz="0"
+                     iyy="${(m/12)*(x*x + z*z)}" iyz="0"
+                     izz="${(m/12)*(x*x + y*y)}" />
+        </inertial>
+    </xacro:macro>
 </robot>

File: src/my_robot_description/urdf/mobile_base.xacro (robot description, xacro)
@@ -16,4 +16,6 @@
             <material name="blue" />
         </visual>
+        <xacro:box_inertia m="5.0" x="${base_length}" y="${base_width}" z="${base_height}"
+                           o_xyz="0.0 0.0 ${base_height/2}" o_rpy="0 0 0" />
     </link>
      <xacro:macro name="wheel_link" params="prefix">

Commit message: included inertia to all

File: src/my_robot_description/urdf/common_properties.xacro (robot description, xacro)
@@ -11,17 +11,26 @@
         <inertial>
             <mass value="${m}" />
-            <orgin xyz="${o_xyz}" rpy="${o_rpy}" />
-            <inertia ixx="${(m/12)*(y*y + z*z)}" ixy="0" ixz="0"
-                     iyy="${(m/12)*(x*x + z*z)}" iyz="0"
-                     izz="${(m/12)*(x*x + y*y)}" />
+            <origin xyz="${o_xyz}" rpy="${o_rpy}" />
+            <inertia ixx="${(m/12) * (y*y + z*z)}" ixy="0" ixz="0"
+                     iyy="${(m/12) * (x*x + z*z)}" iyz="0"
+                     izz="${(m/12) * (x*x + y*y)}" />
         </inertial>
     </xacro:macro>
-    <xacro:macro name="wheel_inertia" params="r l w_xyz w_rpy">
+    <xacro:macro name="cylinder_inertia" params="m r l o_xyz o_rpy">
         <inertial>
             <mass value="${m}" />
-            <orgin xyz="${o_xyz}" rpy="${o_rpy}" />
-            <inertia ixx="${(m/12)*(y*y + z*z)}" ixy="0" ixz="0"
-                     iyy="${(m/12)*(x*x + z*z)}" iyz="0"
-                     izz="${(m/12)*(x*x + y*y)}" />
+            <origin xyz="${o_xyz}" rpy="${o_rpy}" />
+            <inertia ixx="${(m/12) * (3*r*r + l*l)}" ixy="0" ixz="0"
+                     iyy="${(m/12) * (3*r*r + l*l)}" iyz="0"
+                     izz="${(m/2) * (r*r)}" />
+        </inertial>
+    </xacro:macro>
+   <xacro:macro name="sphere_inertia" params="m r o_xyz o_rpy">
+        <inertial>
+            <mass value="${m}" />
+            <origin xyz="${o_xyz}" rpy="${o_rpy}" />
+            <inertia ixx="${(2/5)*m*r*r}" ixy="0" ixz="0"
+                     iyy="${(2/5)*m*r*r}" iyz="0"
+                     izz="${(2/5)*m*r*r}" />
         </inertial>
     </xacro:macro>

File: src/my_robot_description/urdf/mobile_base.xacro (robot description, xacro)
@@ -13,9 +13,9 @@
                 <box size="${base_length} ${base_width} ${base_height}"/>
             </geometry>
-            <origin xyz="0.0 0.0 ${base_height/2}" rpy="0.0 0.0 0.0"/>
+            <origin xyz="0.0 0.0 ${base_height/2.0}" rpy="0.0 0.0 0.0"/>
             <material name="blue" />
         </visual>
         <xacro:box_inertia m="5.0" x="${base_length}" y="${base_width}" z="${base_height}"
-                           o_xyz="0.0 0.0 ${base_height/2}" o_rpy="0 0 0" />
+                           o_xyz="0.0 0.0 ${base_height / 2.0}" o_rpy="0.0 0.0 0.0" />
     </link>
      <xacro:macro name="wheel_link" params="prefix">
@@ -28,4 +28,6 @@
                <material name="grey"/>
             </visual>
+            <xacro:cylinder_inertia m="1.0" r="${wheel_radius}" l="${wheel_length}"
+                           o_xyz="0.0 0.0 0.0" o_rpy="${pi / 2.0} 0.0 0.0" />
         </link>
     </xacro:macro>
@@ -60,4 +62,5 @@
             <material name="grey"/>
         </visual>
+        <xacro:sphere_inertia m="0.5" r="${wheel_radius/2}" o_xyz="0.0 0.0 0.0" o_rpy="0.0 0.0 0.0" />
     </link>
 <!-- Joints -->

Commit message: working on it

File: src/my_robot_description/urdf/common_properties.xacro (robot description, xacro)
@@ -7,4 +7,10 @@
     <material name="grey">
         <color rgba="0.5 0.5 0.5 1" />  <!-- Grey -->
+    </material>
+    <material name="orange">
+        <color rgba="1 0.5 0 1" />      <!-- Orange -->
+    </material>
+    <material name="yellow">
+        <color rgba="1 1 0 1" />      <!-- Yellow -->
     </material>
     <xacro:macro name="box_inertia" params="m x y z o_xyz o_rpy">
