Commit message: Added a arm

File: src/my_robot_description/urdf/arm.xacro (robot description, xacro)
@@ -6,4 +6,6 @@
     <xacro:property name="forearm_radius" value="0.02"/>
     <xacro:property name="forearm_length" value="0.3"/>
+    <xacro:property name="hand_radius" value="0.02"/>
+    <xacro:property name="hand_length" value="0.3"/>
     <link name="arm_base_link">
         <visual>
@@ -20,6 +22,15 @@
             <cylinder radius="${forearm_radius}" length="${forearm_length}"/>
            </geometry>
-           <origin xyz="0 0 ${arm_base_height+(forearm_length/2)}" rpy="0 0 0"/>
+           <origin xyz="0 0 ${(forearm_length/2)}" rpy="0 0 0"/>
            <material name="yellow"/>
+        </visual>
+    </link>
+     <link name="hand_link">
+        <visual>
+           <geometry>
+            <cylinder radius="${hand_radius}" length="${hand_length}"/>
+           </geometry>
+           <origin xyz="0 0 ${(hand_length/2)}" rpy="0 0 0"/>
+           <material name="orange"/>
         </visual>
     </link>
@@ -28,5 +39,12 @@
         <child link="forearm_link"/>
         <origin xyz="0 0 ${arm_base_height}" rpy="0 0 0"/>
-        <axis xyz="1 0 0"/>
+        <axis xyz="0 1 0"/>
+        <limit lower="0" upper="${pi/2}" effort="100" velocity="100"/>
+    </joint>
+     <joint name="forearm_hand_joint" type="revolute">
+        <parent link="forearm_link"/>
+        <child link="hand_link"/>
+        <origin xyz="0 0 ${forearm_length}" rpy="0 0 0"/>
+        <axis xyz="0 1 0"/>
         <limit lower="0" upper="${pi/2}" effort="100" velocity="100"/>
     </joint>

Commit message: Added inertia

File: src/my_robot_description/urdf/arm.xacro (robot description, xacro)
@@ -11,27 +11,51 @@
         <visual>
            <geometry>
-            <box size="${arm_base_length} ${arm_base_width} ${arm_base_height}"/>
+                <box size="${arm_base_length} ${arm_base_width} ${arm_base_height}"/>
            </geometry>
            <origin xyz="0 0 ${arm_base_height/2}" rpy="0 0 0"/>
            <material name="orange"/>
         </visual>
+        <collision>
+            <geometry>
+                <box size="${arm_base_length} ${arm_base_width} ${arm_base_height}"/>
+           </geometry>
+           <origin xyz="0 0 ${arm_base_height/2}" rpy="0 0 0"/>
+        </collision>
+        <xacro:box_inertia m="0.5" x="${arm_base_length}" y="${arm_base_width}" z="${arm_base_height}"
+                            o_xyz="0 0 ${arm_base_height/2}" o_rpy="0 0 0"/>
     </link>
     <link name="forearm_link">
         <visual>
            <geometry>
-            <cylinder radius="${forearm_radius}" length="${forearm_length}"/>
+                <cylinder radius="${forearm_radius}" length="${forearm_length}"/>
            </geometry>
            <origin xyz="0 0 ${(forearm_length/2)}" rpy="0 0 0"/>
            <material name="yellow"/>
         </visual>
+        <collision>
+            <geometry>
+                <cylinder radius="${forearm_radius}" length="${forearm_length}"/>
+           </geometry>
+           <origin xyz="0 0 ${(forearm_length/2)}" rpy="0 0 0"/>
+        </collision>
+        <xacro:cylinder_inertia m="0.3" r="${forearm_radius}" l="${forearm_length}"
+                                o_xyz="0 0 ${(forearm_length/2)}" o_rpy="0 0 0"/>
     </link>
      <link name="hand_link">
         <visual>
            <geometry>
-            <cylinder radius="${hand_radius}" length="${hand_length}"/>
+                <cylinder radius="${hand_radius}" length="${hand_length}"/>
            </geometry>
            <origin xyz="0 0 ${(hand_length/2)}" rpy="0 0 0"/>
            <material name="orange"/>
         </visual>
+        <collision>
+            <geometry>
+                <cylinder radius="${hand_radius}" length="${hand_length}"/>
+           </geometry>
+           <origin xyz="0 0 ${(hand_length/2)}" rpy="0 0 0"/>
+        </collision>
+        <xacro:cylinder_inertia m="0.3" r="${hand_radius}" l="${hand_length}"
+                                o_xyz="0 0 ${(hand_length/2)}" o_rpy="0 0 0"/>
     </link>
     <joint name="arm_base_forearm_joint" type="revolute">

Commit message: Added friction and damping

File: src/my_robot_description/urdf/arm.xacro (robot description, xacro)
@@ -65,4 +65,5 @@
         <axis xyz="0 1 0"/>
         <limit lower="0" upper="${pi/2}" effort="100" velocity="100"/>
+        <dynamics friction="0.3" damping="0.3"/>
     </joint>
      <joint name="forearm_hand_joint" type="revolute">
@@ -72,4 +73,5 @@
         <axis xyz="0 1 0"/>
         <limit lower="0" upper="${pi/2}" effort="100" velocity="100"/>
+        <dynamics friction="0.3" damping="0.3"/>
     </joint>
 </robot>
