Commit message: XACRO Properties testing

File: src/my_robot_description/urdf/my_robot.urdf.xacro (robot description, xacro)
@@ -1,10 +1,15 @@
 <?xml version="1.0"?>
-<robot name="my_robot">
+<robot name="my_robot" xmlns:xacro="http://www.ros.org/wiki/xacro">
+    <xacro:property name="base_length" value="0.6" />
+    <xacro:property name="base_width" value="0.4" />
+    <xacro:property name="base_height" value="0.2" />
+    <xacro:property name="wheel_radius" value="0.1" />
+    <xacro:property name="wheel_length" value="0.05" />
 <!-- Material -->
     <material name="blue">
-        <color rgba="0 0 0.5 1" />
+        <color rgba="0 0 0.5 1" />      <!-- Blue -->
     </material>
     <material name="grey">
-        <color rgba="0.5 0.5 0.5 1" />
+        <color rgba="0.5 0.5 0.5 1" />  <!-- Grey -->
     </material>
 <!-- Links -->
@@ -13,7 +18,7 @@
         <visual>
             <geometry>
-                <box size="0.6 0.4 0.2"/>
+                <box size="${base_length} ${base_width} ${base_height}"/>
             </geometry>
-            <origin xyz="0.0 0.0 0.1" rpy="0.0 0.0 0.0"/>
+            <origin xyz="0.0 0.0 ${base_height/2}" rpy="0.0 0.0 0.0"/>
             <material name="blue" />
         </visual>
@@ -22,7 +27,7 @@
         <visual>
             <geometry>
-                <cylinder radius="0.1" length="0.05"/>
+                <cylinder radius="${wheel_radius}" length="${wheel_length}"/>
             </geometry>
-            <origin xyz="0.0 0.0 0.0" rpy="1.57 0.0 0.0"/>
+            <origin xyz="0.0 0.0 0.0" rpy="${pi / 2.0} 0.0 0.0"/>
             <material name="grey"/>
         </visual>
@@ -31,7 +36,7 @@
         <visual>
             <geometry>
-                <cylinder radius="0.1" length="0.05"/>
+                <cylinder radius="${wheel_radius}" length="${wheel_length}"/>
             </geometry>
-            <origin xyz="0.0 0.0 0.0" rpy="1.57 0.0 0.0"/>
+            <origin xyz="0.0 0.0 0.0" rpy="${pi/2.0} 0.0 0.0"/>
             <material name="grey"/>
         </visual>
@@ -40,5 +45,5 @@
         <visual>
             <geometry>
-                <sphere radius="0.05"/>
+                <sphere radius="${wheel_radius/2}"/>
             </geometry>
             <origin xyz="0.0 0.0 0.0" rpy="0.0 0.0 0.0"/>
@@ -50,5 +55,5 @@
         <parent link="base_footprint"/>
         <child link="base_link"/>
-        <origin xyz="0.0 0.0 0.1" rpy="0.0 0.0 0.0"/>
+        <origin xyz="0.0 0.0 ${wheel_radius}" rpy="0.0 0.0 0.0"/>
     </joint>
     <joint name="base_right_wheel_joint" type="continuous">
@@ -56,5 +61,5 @@
         <child link="right_wheel_link"/>
         <axis xyz="0 1 0"/>
-        <origin xyz="-0.15 -0.225 0" rpy="0 0 0"/>
+        <origin xyz="${-base_length/4.0} ${-(base_width + wheel_length )/2} 0" rpy="0 0 0"/>
     </joint>
     <joint name="base_left_wheel_joint" type="continuous">
@@ -62,5 +67,5 @@
         <child link="left_wheel_link"/>
         <axis xyz="0 1 0"/>
-        <origin xyz="-0.15 0.225 0" rpy="0 0 0"/>
+        <origin xyz="${-base_length/4.0} ${(base_width + wheel_length )/2} 0" rpy="0 0 0"/>
     </joint>
     <joint name="base_caster_wheel_joint" type="fixed">
@@ -68,5 +73,5 @@
         <child link="caster_wheel_link"/>
         <axis xyz="0 1 0"/>
-        <origin xyz="0.2 0.0 -0.05" rpy="0 0 0"/>
+        <origin xyz="${base_length/3.0} 0.0 ${-wheel_radius/2}" rpy="0 0 0"/>
     </joint>
 </robot>

Commit message: XACRO:MACRO  Used

File: src/my_robot_description/urdf/my_robot.urdf.xacro (robot description, xacro)
@@ -24,4 +24,18 @@
         </visual>
     </link>
+     <xacro:macro name="wheel_link" params="prefix">
+        <link name="${prefix}_wheel_link">
+            <visual>
+                <geometry>
+                    <cylinder radius="${wheel_radius}" length="${wheel_length}"/>
+                </geometry>
+                <origin xyz="0.0 0.0 0.0" rpy="${pi / 2.0} 0.0 0.0"/>
+               <material name="grey"/>
+            </visual>
+        </link>
+    </xacro:macro>
+    <xacro:wheel_link prefix="right" />
+    <xacro:wheel_link prefix="left" />
+<!-- Normal link and the above is the XACRO:MACRO Feature
     <link name="right_wheel_link">
         <visual>
@@ -42,4 +56,5 @@
         </visual>
     </link>
+-->
     <link name="caster_wheel_link">
         <visual>

Commit message: Urdf file got separated using xacro

File: src/my_robot_description/urdf/my_robot.urdf.xacro (robot description, xacro)
@@ -1,92 +1,5 @@
 <?xml version="1.0"?>
 <robot name="my_robot" xmlns:xacro="http://www.ros.org/wiki/xacro">
-    <xacro:property name="base_length" value="0.6" />
-    <xacro:property name="base_width" value="0.4" />
-    <xacro:property name="base_height" value="0.2" />
-    <xacro:property name="wheel_radius" value="0.1" />
-    <xacro:property name="wheel_length" value="0.05" />
-<!-- Material -->
-    <material name="blue">
-        <color rgba="0 0 0.5 1" />      <!-- Blue -->
-    </material>
-    <material name="grey">
-        <color rgba="0.5 0.5 0.5 1" />  <!-- Grey -->
-    </material>
-<!-- Links -->
-    <link name="base_footprint" />
-    <link name="base_link">
-        <visual>
-            <geometry>
-                <box size="${base_length} ${base_width} ${base_height}"/>
-            </geometry>
-            <origin xyz="0.0 0.0 ${base_height/2}" rpy="0.0 0.0 0.0"/>
-            <material name="blue" />
-        </visual>
-    </link>
-     <xacro:macro name="wheel_link" params="prefix">
-        <link name="${prefix}_wheel_link">
-            <visual>
-                <geometry>
-                    <cylinder radius="${wheel_radius}" length="${wheel_length}"/>
-                </geometry>
-                <origin xyz="0.0 0.0 0.0" rpy="${pi / 2.0} 0.0 0.0"/>
-               <material name="grey"/>
-            </visual>
-        </link>
-    </xacro:macro>
-    <xacro:wheel_link prefix="right" />
-    <xacro:wheel_link prefix="left" />
-<!-- Normal link and the above is the XACRO:MACRO Feature
-    <link name="right_wheel_link">
-        <visual>
-            <geometry>
-                <cylinder radius="${wheel_radius}" length="${wheel_length}"/>
-            </geometry>
-            <origin xyz="0.0 0.0 0.0" rpy="${pi / 2.0} 0.0 0.0"/>
-            <material name="grey"/>
-        </visual>
-    </link>
-    <link name="left_wheel_link">
-        <visual>
-            <geometry>
-                <cylinder radius="${wheel_radius}" length="${wheel_length}"/>
-            </geometry>
-            <origin xyz="0.0 0.0 0.0" rpy="${pi/2.0} 0.0 0.0"/>
-            <material name="grey"/>
-        </visual>
-    </link>
--->
-    <link name="caster_wheel_link">
-        <visual>
-            <geometry>
-                <sphere radius="${wheel_radius/2}"/>
-            </geometry>
-            <origin xyz="0.0 0.0 0.0" rpy="0.0 0.0 0.0"/>
-            <material name="grey"/>
-        </visual>
-    </link>
-<!-- Joints -->
-    <joint name="base_joint" type="fixed">
-        <parent link="base_footprint"/>
-        <child link="base_link"/>
-        <origin xyz="0.0 0.0 ${wheel_radius}" rpy="0.0 0.0 0.0"/>
-    </joint>
-    <joint name="base_right_wheel_joint" type="continuous">
-        <parent link="base_link"/>
-        <child link="right_wheel_link"/>
-        <axis xyz="0 1 0"/>
-        <origin xyz="${-base_length/4.0} ${-(base_width + wheel_length )/2} 0" rpy="0 0 0"/>
-    </joint>
-    <joint name="base_left_wheel_joint" type="continuous">
-        <parent link="base_link"/>
-        <child link="left_wheel_link"/>
-        <axis xyz="0 1 0"/>
-        <origin xyz="${-base_length/4.0} ${(base_width + wheel_length )/2} 0" rpy="0 0 0"/>
-    </joint>
-    <joint name="base_caster_wheel_joint" type="fixed">
-        <parent link="base_link"/>
-        <child link="caster_wheel_link"/>
-        <axis xyz="0 1 0"/>
-        <origin xyz="${base_length/3.0} 0.0 ${-wheel_radius/2}" rpy="0 0 0"/>
-    </joint>
+    <xacro:include filename="common_properties.xacro" />
+    <xacro:include filename="mobile_base.xacro" />
 </robot>

Commit message: combained all

File: src/my_robot_description/urdf/my_robot.urdf.xacro (robot description, xacro)
@@ -4,5 +4,11 @@
     <xacro:include filename="mobile_base.xacro" />
     <xacro:include filename="mobile_base_gazebo.xacro" />
+    <xacro:include filename="arm.xacro" />
+    <xacro:include filename="arm_gazebo.xacro" />
     <xacro:include filename="camera.xacro" />
-    <xacro:include filename="arm.xacro" />
+    <joint name="mobile_base_arm_joint" type="fixed">
+        <parent link="base_link"/>
+        <child link="arm_base_link"/>
+        <origin xyz="${base_length/4} 0 ${base_height}" rpy="0 0 0"/>
+    </joint>
 </robot>
